File: pcb/KiCad Schematic.kicad_pcb (KiCad board)
At the start: 4 copper layers, 70 x 100 mm, 161 parts, among them IC1 AP63205WU-7, IC2 ATSAMD51J19A-MU, IC4 TMC5160A-TA-T, IC6 TMC5160A-TA-T, IC7 TMC5160A-TA-T, J12 Conn_01x03, J13 Conn_01x10, J14 Conn_01x04, J15 Conn_01x03, J16 Conn_01x03, J17 Hole, J18 Hole, J19 Hole, J2 Conn_01x02, J20 Hole, J21 Conn_01x02, J22 Conn_01x06, J23 Conn_01x04, J24 Conn_01x04, J25 Conn_01x05, J26 Conn_01x05, J27 Conn_01x05, J3 47346-0001, J6 20021121-00010C4LF, J8 Conn_01x02, J9 Conn_01x02, Q13 FDMC8030, Q14 FDMC8030, Q15 FDMC8030, Q16 FDMC8030, Q17 FDMC8030, Q18 FDMC8030, Q19 FDMC8030, Q20 FDMC8030, Q5 FDMC8030, Q6 FDMC8030, Q7 FDMC8030, Q8 FDMC8030, U3 AP2112K-3.3, Y1 LFXTAL009678REEL

Commit message: final 1.0 stuff and first pass arduino library
Parts:
- removed J12: Conn_01x03, Connector_PinHeader_2.54mm:PinHeader_1x03_P2.54mm_Vertical
- removed J21: Conn_01x02, Connector_PinHeader_2.54mm:PinHeader_1x02_P2.54mm_Vertical
- added C12: 100nF, Capacitor_SMD:C_0603_1608Metric, F.Cu at (83.4, 158.7)
- added C13: 100nF, Capacitor_SMD:C_0603_1608Metric, F.Cu at (80.7, 163.2)
- added C14: 2.2uF, Capacitor_SMD:C_1206_3216Metric, F.Cu at (81.4, 157.9)
- added C15: 470nF, Capacitor_SMD:C_0603_1608Metric, F.Cu at (80.7, 161.6)
- added C16: 22nF, Capacitor_SMD:C_0603_1608Metric, F.Cu at (83.0, 162.4)
- added C17: 100nF, Capacitor_SMD:C_0603_1608Metric, F.Cu at (90.2, 153.1)
- added C18: 100nF, Capacitor_SMD:C_0603_1608Metric, F.Cu at (90.2, 167.8)
- added C19: 47uF, Capacitor_SMD:CP_Elec_6.3x7.7, F.Cu at (80.8, 168.8)
- added C20: 100nF, Capacitor_SMD:C_0603_1608Metric, F.Cu at (95.0, 159.8)
- added C21: 100nF, Capacitor_SMD:C_0603_1608Metric, F.Cu at (111.8, 162.3)
- added C22: 100nF, Capacitor_SMD:C_0603_1608Metric, F.Cu at (114.5, 157.7)
- added C23: 2.2uF, Capacitor_SMD:C_1206_3216Metric, F.Cu at (113.8, 163.0)
- added C24: 470nF, Capacitor_SMD:C_0603_1608Metric, F.Cu at (114.4, 159.3)
- added C26: 22nF, Capacitor_SMD:C_0603_1608Metric, F.Cu at (112.2, 158.6)
- added C27: 100nF, Capacitor_SMD:C_0603_1608Metric, F.Cu at (105.0, 167.8)
- added C42: 100nF, Capacitor_SMD:C_0603_1608Metric, F.Cu at (105.0, 153.1)
- added C49: 47uF, Capacitor_SMD:CP_Elec_6.3x7.7, F.Cu at (114.3, 152.1)
- added C50: 100nF, Capacitor_SMD:C_0603_1608Metric, F.Cu at (100.2, 161.2)
- added G***: LOGO, imgs:smol_logo, F.Cu at (70.4, 146.3)
- added G***: LOGO, imgs:logo, B.Cu at (93.6, 120.5)
- added J1: Conn_01x04, Connector_PinHeader_2.54mm:PinHeader_1x04_P2.54mm_Vertical, F.Cu at (86.5, 171.2)
- added J4: Conn_01x04, Connector_PinHeader_2.54mm:PinHeader_1x04_P2.54mm_Vertical, F.Cu at (86.5, 149.7)
- added J5: Conn_01x04, Connector_PinHeader_2.54mm:PinHeader_1x04_P2.54mm_Vertical, F.Cu at (108.7, 149.7)
- added J7: Conn_01x04, Connector_PinHeader_2.54mm:PinHeader_1x04_P2.54mm_Vertical, F.Cu at (108.6, 171.2)
- added R10: 0R2, Resistor_SMD:R_0805_2012Metric, F.Cu at (107.8, 153.6)
- added R11: 0R2, Resistor_SMD:R_0805_2012Metric, F.Cu at (102.0, 167.3)
- added R12: 0R2, Resistor_SMD:R_0805_2012Metric, F.Cu at (107.8, 167.3)
- added R3: 2R2, Resistor_SMD:R_0603_1608Metric, F.Cu at (79.4, 158.7)
- added R4: 0R2, Resistor_SMD:R_0805_2012Metric, F.Cu at (93.1, 167.3)
- added R5: 0R2, Resistor_SMD:R_0805_2012Metric, F.Cu at (87.3, 167.3)
- added R6: 0R2, Resistor_SMD:R_0805_2012Metric, F.Cu at (93.1, 153.7)
- added R7: 0R2, Resistor_SMD:R_0805_2012Metric, F.Cu at (87.3, 153.7)
- added R8: 2R2, Resistor_SMD:R_0603_1608Metric, F.Cu at (115.8, 162.2)
- added R9: 0R2, Resistor_SMD:R_0805_2012Metric, F.Cu at (102.0, 153.6)
- added U1: TMC2041-LA, Package_DFN_QFN:QFN-48-1EP_7x7mm_P0.5mm_EP5.3x5.3mm, F.Cu at (89.9, 160.5)
- added U2: TMC2041-LA, Package_DFN_QFN:QFN-48-1EP_7x7mm_P0.5mm_EP5.3x5.3mm, F.Cu at (105.2, 160.4)
- IC2: footprint Package_DFN_QFN:QFN-64-1EP_9x9mm_P0.5mm_EP6x6mm_ThermalVias -> Package_DFN_QFN:QFN-64-1EP_9x9mm_P0.5mm_EP6x6mm
- J2: value Conn_01x02 -> 691313710002; footprint Connector_BarrelJack:BarrelJack_Wuerth_6941xx301002 -> SamacSys_Parts:691313710002
- J8: value Conn_01x02 -> Conn_01x05; footprint Connector_PinHeader_2.54mm:PinHeader_1x02_P2.54mm_Vertical -> Connector_PinHeader_2.54mm:PinHeader_1x05_P2.54mm_Vertical
- J9: value Conn_01x02 -> Conn_01x04; footprint Connector_PinHeader_2.54mm:PinHeader_1x02_P2.54mm_Vertical -> Connector_PinHeader_2.54mm:PinHeader_1x04_P2.54mm_Vertical
- R16, R18: value 10k -> 2k2
- moved R17 119.0 mm to (66.2, 129.6)
- moved D1 116.2 mm to (66.2, 131.3), turned to 180 degrees
- moved C31 96.8 mm to (61.9, 167.1)
- moved J9 96.4 mm to (66.9, 155.7)
- moved J22 90.2 mm to (61.8, 150.6)
- moved J16 85.4 mm to (59.0, 203.2), turned to 90 degrees
- moved J15 81.0 mm to (59.0, 200.6), turned to 90 degrees
- moved D2 72.4 mm to (81.1, 203.7), turned to 180 degrees
- moved J8 69.0 mm to (67.7, 203.2), turned to 90 degrees
- moved R20 65.5 mm to (81.1, 202.1)
- moved R1 64.2 mm to (80.3, 199.0), turned to 90 degrees
- moved C3 63.4 mm to (78.7, 199.0), turned to 270 degrees
- moved R19 62.7 mm to (77.1, 199.0), turned to 90 degrees
- moved S1 60.3 mm to (71.8, 198.8), turned to 180 degrees
- moved J3 38.4 mm to (49.5, 178.0)
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Connections:
- IC2 pad 10: /GEN3 -> /GPIO4
- IC2 pad 11: /GEN4 -> /GPIO5
- IC2 pad 12: /GEN5 -> /D5D6_EN
- IC2 pad 13: /GEN6 -> /D5_STEP
- IC2 pad 14: /GEN7 -> /D5_DIR
- IC2 pad 15: /GEN8 -> /D6_STEP
- IC2 pad 16: /GEN9 -> /D6_DIR
- IC2 pad 19: /D2_DIR -> /D3D4_CS
- IC2 pad 20: /D2_STEP -> /D3D4_EN
- IC2 pad 23: /D2_CS -> /D3_STEP
- IC2 pad 24: /D2_EN -> /D3_DIR
- IC2 pad 25: Net-(IC2-Pad25) -> /D4_STEP
- IC2 pad 26: Net-(IC2-Pad26) -> /D4_DIR
- IC2 pad 27: /D1_EN -> /D5D6_CS
- IC2 pad 28: /D1_CS -> /D1_DIR
- IC2 pad 32: /D1_DIR -> /D1_CS
- IC2 pad 35: Net-(IC2-Pad35) -> /D1_EN
- IC2 pad 37: /D0_EN -> /D2_DIR
- IC2 pad 38: /D0_CS -> /D2_STEP
- IC2 pad 41: /D0_STEP -> /D2_CS
- IC2 pad 42: /D0_DIR -> /D2_EN
- IC2 pad 5: /GEN0 -> /GPIO1
- IC2 pad 59: Net-(IC2-Pad59) -> /D0_DIR
- IC2 pad 6: /GEN1 -> /GPIO2
- IC2 pad 60: Net-(IC2-Pad60) -> /D0_STEP
- IC2 pad 61: Net-(IC2-Pad61) -> /D0_CS
- IC2 pad 62: Net-(IC2-Pad62) -> /D0_EN
- IC2 pad 9: /GEN2 -> /GPIO3
- J13 pad 1: /GEN0 -> Net-(J13-Pad1)
- J13 pad 10: /GEN9 -> /CAN_RX
- J13 pad 2: /GEN1 -> /MISO
- J13 pad 3: /GEN2 -> /MOSI
- J13 pad 4: /GEN3 -> /SCK
- J13 pad 5: /GEN4 -> /SDA
- J13 pad 6: /GEN5 -> /SCL
- J13 pad 7: /GEN6 -> /TX
- J13 pad 8: /GEN7 -> /RX
- J13 pad 9: /GEN8 -> /CAN_TX
- J8 pad 1: /CAN_TX -> /GPIO1
- J8 pad 2: /CAN_RX -> /GPIO2
- J9 pad 1: /SDA -> +5V
- J9 pad 2: /SCL -> GND
- R20 pad 2: /GEN14 -> /GPIO5
Routing:
- net +3V3: track 39.2 -> 329.1 mm, vias 0 -> 17
- net +VDC: track 107.3 -> 356.0 mm, vias 36 -> 52
- net +5V: track 12.5 -> 188.8 mm, vias 0 -> 3
- net /MOSI: track 10.6 -> 178.2 mm, vias 0 -> 9
- net /MISO: track 9.24 -> 176.1 mm, vias 0 -> 8
- net /SCK: track 6.02 -> 167.0 mm, vias 0 -> 10
- net GND: track 133.5 -> 294.1 mm, vias 43 -> 106
- net /D1_EN: track 15.2 -> 98.4 mm
- net /D5D6_CS: track 0.00 -> 71.4 mm
- net /D5D6_EN: track 0.00 -> 69.4 mm
- net /D5_STEP: track 0.00 -> 67.4 mm
- net /D2_STEP: track 0.00 -> 67.1 mm
- net /D2_DIR: track 0.00 -> 66.7 mm
- net /D1_CS: track 0.00 -> 65.5 mm, vias 0 -> 2
- net /D5_DIR: track 0.00 -> 65.4 mm
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- added copper zone on F.Cu, net +3V3
Other:
- board text added: "'"
- board text added: "0"
- board text added: "1"
- board text added: "2"
- board text added: "3"
- board text added: "3V3"
- board text added: "4"
- board text added: "5V"
- board text added: "7V-24V"
- board text added: "C|RX"
- board text added: "C|TX"
- board text added: "ENC0"
- board text added: "ENC1"
- board text added: "ENC2"
- board text added: "ENCODER I2C BUS"
- board text added: "GND"
- board text added: "LOL"
- board text added: "MISO"
- board text added: "MOSI"
- board text added: "RX"
- board text added: "S0"
- board text added: "S1"
- board text added: "SCK"
- board text added: "SCL"
- board text added: "SDA"
- board text added: "SIG"
- board text added: "STEP0"
- board text added: "STEP1"
- board text added: "STEP2"
- board text added: "STEP3"
- board text added: "STEP4"
- board text added: "STEP5"
- board text added: "STEP6"
- board text added: "TX"
- board text added: "V1.0"
- board text added: "VDC"
