File: pcb/KiCad Schematic.sch (KiCad schematic (older format))
At the start: 53 parts, among them IC1 AP63205WU-7, IC2 ATSAMD51J19A-MU, J12 Conn_01x03, J13 Conn_01x10, J15 Conn_01x03, J16 Conn_01x03, J17 Hole, J18 Hole, J19 Hole, J2 Conn_01x02, J20 Hole, J21 Conn_01x02, J22 Conn_01x06, J3 47346-0001, J6 20021121-00010C4LF, J8 Conn_01x02, J9 Conn_01x02, U3 AP2112K-3.3, Y1 LFXTAL009678REEL

Commit message: final 1.0 stuff and first pass arduino library
Parts:
- removed J12: Conn_01x03, Connector_PinHeader_2.54mm:PinHeader_1x03_P2.54mm_Vertical, symbol Connector_Generic:Conn_01x03
- removed J2: Conn_01x02, Connector_BarrelJack:BarrelJack_Wuerth_6941xx301002, symbol Connector_Generic:Conn_01x02
- removed J21, J8, J9: Conn_01x02, Connector_PinHeader_2.54mm:PinHeader_1x02_P2.54mm_Vertical, symbol Connector_Generic:Conn_01x02
- added J2: 691313710002, 691313710002, symbol SamacSys_Parts:691313710002
- added J8: Conn_01x05, Connector_PinHeader_2.54mm:PinHeader_1x05_P2.54mm_Vertical, symbol Connector_Generic:Conn_01x05
- added J9: Conn_01x04, Connector_PinHeader_2.54mm:PinHeader_1x04_P2.54mm_Vertical, symbol Connector_Generic:Conn_01x04
- R16, R18: value 10k -> 2k2
Connections:
- net +5V: now also J9.1 (Pin_1)
- net +VDC: now also J2.1
- net CAN_RX: now also J13.10 (Pin_10)
- net CAN_TX: now also J13.9 (Pin_9)
- net D0_CS: now also IC2.61 (PB00); no longer IC2.38 (PA19)
- net D0_DIR: now also IC2.59 (PB30); no longer IC2.42 (PA21)
- net D0_EN: now also IC2.62 (PB01); no longer IC2.37 (PA18)
- net D0_STEP: now also IC2.60 (PB31); no longer IC2.41 (PA20)
- net D1_CS: now also IC2.32 (PA15); no longer IC2.28 (PB15)
- net D1_DIR: now also IC2.28 (PB15); no longer IC2.32 (PA15)
- net D1_EN: now also IC2.35 (PA16); no longer IC2.27 (PB14)
- net D2_CS: now also IC2.41 (PA20); no longer IC2.23 (PB10)
- net D2_DIR: now also IC2.37 (PA18); no longer IC2.19 (PA10)
- net D2_EN: now also IC2.42 (PA21); no longer IC2.24 (PB11)
- net D2_STEP: now also IC2.38 (PA19); no longer IC2.20 (PA11)
- net GND: now also J2.2, J9.2 (Pin_2)
- net MISO: now also J13.2 (Pin_2)
- net MOSI: now also J13.3 (Pin_3)
- net RX: now also J13.8 (Pin_8)
- net SCK: now also J13.4 (Pin_4)
- net SCL: now also J13.6 (Pin_6), J9.4 (Pin_4)
- net SDA: now also J13.5 (Pin_5), J9.3 (Pin_3)
- net TX: now also J13.7 (Pin_7)
- net D4_STEP: now reaches IC2.25 (PB12)
- net D4_DIR: now reaches IC2.26 (PB13)
- net GEN0: no longer names the net of J13.1 (Pin_1)
- net GEN0: no longer IC2.5 (PB04)
- net GEN1 renamed GPIO2
- net GPIO2: now also J8.2 (Pin_2); no longer J13.2 (Pin_2)
- net GEN14 renamed GPIO5
- net GPIO5: now also IC2.11 (PB08), J8.5 (Pin_5)
- net GEN2 renamed GPIO3
- net GPIO3: now also J8.3 (Pin_3); no longer J13.3 (Pin_3)
- net GEN3 renamed GPIO4
- net GPIO4: now also J8.4 (Pin_4); no longer J13.4 (Pin_4)
- removed net GEN4: IC2.11 (PB08), J13.5 (Pin_5)
- net GEN5 renamed D5D6_EN
- net D5D6_EN: no longer J13.6 (Pin_6)
- net GEN6 renamed D5_STEP
- net D5_STEP: no longer J13.7 (Pin_7)
- net GEN7 renamed D5_DIR
- net D5_DIR: no longer J13.8 (Pin_8)
- net GEN8 renamed D6_STEP
- net D6_STEP: no longer J13.9 (Pin_9)
- net GEN9 renamed D6_DIR
- net D6_DIR: no longer J13.10 (Pin_10)
- new net D3D4_CS: IC2.19 (PA10)
- new net D3D4_EN: IC2.20 (PA11)
- new net D3_DIR: IC2.24 (PB11)
- new net D3_STEP: IC2.23 (PB10)
- new net D5D6_CS: IC2.27 (PB14)
- new net GPIO1: IC2.5 (PB04), J8.1 (Pin_1)
- no-connect marks 0 -> 7
Other:
- note added: "STEPPERS"
- note removed: "STEPPER 0"
